File: ESP32-C3-MINI-1-N4-DEVKIT_V2.kicad_sch (KiCad schematic)
At the start: 19 parts, among them J1 USB_C_Receptacle_USB2.0, Q1 MMSS8050, SW1 TL6330AF200Q, U1 ESP32-C3-MINI-1, U2 CP2102N-Axx-xQFN28, U3 AZ1117CH-3.3TRG1

Commit message: power and buttons done in schem
todo: C3 mini + CP2102 the layout can begin
Parts:
- removed C4: 4.7uF, Capacitor_Tantalum_SMD:CP_EIA-3216-18_Kemet-A, symbol Device:C_Polarized_Small
- removed C5: 10uF, Capacitor_Tantalum_SMD:CP_EIA-3216-18_Kemet-A, symbol Device:C_Polarized_Small
- added C10, C9: 22pF, Capacitor_SMD:C_0603_1608Metric, symbol Device:C_Small
- added C4, C5, C8: 10uF, Capacitor_SMD:C_0805_2012Metric, symbol Device:C_Small
- added C6, C7, C? (x2): 0.1uF, Capacitor_SMD:C_0603_1608Metric, symbol Device:C_Small
- added D1: RED_LED, Diode_SMD:D_0603_1608Metric, symbol Device:LED_Small
- added Q2: MMSS8050, Package_TO_SOT_SMD:SOT-23, symbol Device:Q_NPN_BEC
- added R10, R11, R12, R13: 0 Ohm, Resistor_SMD:R_0603_1608Metric, symbol Device:R_Small
- added R7: 4.7k Ohm, Resistor_SMD:R_0603_1608Metric, symbol Device:R_Small
- added R8, R9: 10k Ohm, Resistor_SMD:R_0603_1608Metric, symbol Device:R_Small
- added SW?: TL6330AF200Q, Button_Switch_SMD:SW_Push_1P1T_NO_CK_KMR2, symbol Switch:SW_MEC_5E
- renumbered D1 to D3
Connections:
- net Earth: now reaches D2.1 (A)
- net Earth: now also J1.A1 (GND), J1.A12 (GND), J1.B1 (GND), J1.B12 (GND), J1.S1 (SHIELD), SW1.1, U3.1 (GND), C10.2, C5.2, C6.2, C7.2, C8.2, C9.2, C?.1, C?.1, D1.1 (K), SW?.1
- net VBUS_5V: now reaches D2.2 (K)
- net VBUS_5V: now also D3.2 (A), J1.A4 (VBUS), J1.A9 (VBUS), J1.B4 (VBUS), J1.B9 (VBUS)
- net D-: now reaches D2.3 (K)
- net D-: now also J1.A7 (D-), J1.B7 (D-), R10.1, R11.1
- net D+: now reaches D2.4 (K)
- net D+: now also J1.A6 (D+), J1.B6 (D+), R12.1, R13.1
- net VDD_5V: now reaches D3.1 (K)
- net VDD_5V: now also U3.3 (VI), C5.1, C6.1, R7.1
- net GPIO9: now reaches SW1.3 (K)
- net GPIO9: now also C?.2, Q2.3 (C)
- net at Q1.1 (B): now also R8.2
- net RTS: now reaches Q1.2 (E)
- net RTS: now also R9.1
- net CHIP_PU: now reaches Q1.3 (C)
- net CHIP_PU: now also C?.2, SW?.3 (K)
- net VDD_3V3: now reaches U3.2 (VO)
- net VDD_3V3: now also C7.1, C8.1
- new net: Q2.1 (B), R9.2
- new net: D1.2 (A), R7.2
- new net DTR: Q2.2 (E), R8.1
- new net GPIO18: C9.1, R11.2
- new net GPIO19: C10.1, R12.2
- new net USB_DN: R10.2
- new net USB_DP: R13.2
- no-connect marks 0 -> 8
Other:
- note added: "3V3 VOLTAGE REGULATION"
- note added: "AUTO-PROGRAM TRANSISTORS"
- note added: "BOOT AND RESET BUTTONS"
- note added: "USB INPUT"
- moved on the sheet: C1, C2, C3, D2, D3, J1, Q1, R1, R2, R3, R4, R5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

Commit message: wired cp2102, started C3 mini
Parts:
- removed U2: CP2102N-Axx-xQFN28, Package_DFN_QFN:QFN-28-1EP_5x5mm_P0.5mm_EP3.35x3.35mm, symbol Interface_USB:CP2102N-Axx-xQFN28
- added C? (x3): 0.1uF, Capacitor_SMD:C_0603_1608Metric, symbol Device:C_Small
- added C?: 1uF, Capacitor_SMD:C_0603_1608Metric, symbol Device:C_Small
- added C? (x3): 10uF, Capacitor_SMD:C_0805_2012Metric, symbol Device:C_Small
- added D?: RX_LED, Diode_SMD:D_0603_1608Metric, symbol Device:LED_Small
- added D?: TX_LED, Diode_SMD:D_0603_1608Metric, symbol Device:LED_Small
- added R? (x2): 10k, Resistor_SMD:R_0603_1608Metric, symbol Device:R_Small
- added R? (x3): 1k, Resistor_SMD:R_0603_1608Metric, symbol Device:R_Small
- added R? (x2): 4.7k, Resistor_SMD:R_0603_1608Metric, symbol Device:R_Small
- added U?: CP2102N-Axx-xQFN24, Package_DFN_QFN:QFN-24-1EP_4x4mm_P0.5mm_EP2.6x2.6mm, symbol Interface_USB:CP2102N-Axx-xQFN24
- D1: value RED_LED -> PWR_LED
- R5: value 22.1k Ohm -> 22.1k
- R6: value 47.5k Ohm -> 47.5k
- R7: value 4.7k Ohm -> 4.7k
Connections:
- net DTR: now also U?.23 (~{DTR})
- net Earth: now also R6.2, U1.1 (GND), U1.11 (GND), U1.14 (GND), U1.2 (GND), U1.36 (GND), C?.2, C?.2, C?.2, C?.2, C?.2, C?.2, C?.2, R?.2, R?.2, R?.2, U?.2 (GND), U?.25 (GND)
- net RTS: now also U?.19 (~{RTS})
- net USB_DN: now also U?.4 (D-)
- net USB_DP: now also U?.3 (D+)
- net VBUS_5V: now also R5.1, C?.1, C?.1, U?.7 (VREGIN)
- net VDD_3V3: now also U1.3 (3V3), C?.1, C?.1, C?.1, C?.1, R?.1, R?.1, R?.2, R?.2, U?.5 (VIO), U?.6 (VDD)
- net RXD: now reaches U1.30 (GPIO20/U0RXD)
- net RXD: now also U?.20 (RXD)
- net TXD: now reaches U1.31 (GPIO21/U0TXD)
- net TXD: now also U?.21 (TXD)
- net at J1.A5 (CC1): now also R?.1
- net at J1.B5 (CC2): now also R?.1
- net at R5.2: now also R6.1, C?.1, U?.8 (VBUS)
- new net: D?.1 (K), U?.13 (~{RXT}/GPIO.1)
- new net: D?.2 (A), R?.1 (x2)
- new net: R?.2, U?.9 (~{RST})
- new net: R?.1, U?.15 (~{SUSPEND})
- new net: D?.1 (K), U?.14 (~{TXT}/GPIO.0)
- new net GPIO8: R?.2
- no-connect marks 8 -> 13
Other:
- note added: "CC1+CC2 Pulldown = Upstream-Facing Port (peripheral)"
- moved on the sheet: C10, C9, D1, R5, R6, R7

Commit message: started layout
Parts:
- removed C2: 0.1uF, Capacitor_SMD:C_0603_1608Metric, symbol Device:C_Small
- removed C3: 1uF, Capacitor_SMD:C_0603_1608Metric, symbol Device:C_Small
- removed C4: 10uF, Capacitor_SMD:C_0805_2012Metric, symbol Device:C_Small
- removed R2: 1k Ohm, Resistor_SMD:R_0603_1608Metric, symbol Device:R_Small
- removed R3: 4.7k Ohm, Resistor_SMD:R_0603_1608Metric, symbol Device:R_Small
- removed R4: 10k Ohm, Resistor_SMD:R_0603_1608Metric, symbol Device:R_Small
- added J2, J3: Conn_01x15, Connector_PinHeader_2.54mm:PinHeader_1x15_P2.54mm_Vertical, symbol Connector_Generic:Conn_01x15
- C1: value 22pF -> 1uF
- R1: value 0 Ohm -> 10k
- R10, R11, R12, R13: value 0 Ohm -> 0
- R8, R9: value 10k Ohm -> 10k
- gave numbers to parts that had none: 20
Connections:
- net CHIP_PU: now also C1.1, R1.2, U1.8 (EN/CHIP_PU), J2.7 (Pin_7)
- net Earth: now also C1.2, J2.1 (Pin_1), J2.12 (Pin_12), J2.15 (Pin_15), J2.6 (Pin_6), J2.8 (Pin_8), J3.1 (Pin_1), J3.12 (Pin_12), J3.15 (Pin_15), J3.4 (Pin_4), J3.7 (Pin_7)
- net GPIO18: now also U1.26 (GPIO18/USB_D-), J3.13 (Pin_13)
- net GPIO19: now also U1.27 (GPIO19/USB_D+), J3.14 (Pin_14)
- net GPIO8: now also U1.22 (GPIO8), J3.6 (Pin_6)
- net GPIO9: now also U1.23 (GPIO9), J3.5 (Pin_5)
- net VBUS_5V: now also J2.13 (Pin_13), J2.14 (Pin_14)
- net VDD_3V3: now also R1.1, J2.2 (Pin_2), J2.3 (Pin_3)
- net GPIO0: now reaches U1.12 (GPIO0/ADC1_CH0/XTAL_32K_P)
- net GPIO0: now also J2.9 (Pin_9)
- net GPIO1: now reaches U1.13 (GPIO1/ADC1_CH1/XTAL_32K_N)
- net GPIO1: now also J2.10 (Pin_10)
- net GPIO10: now reaches U1.16 (GPIO10)
- net GPIO10: now also J2.11 (Pin_11)
- net GPIO4: now reaches U1.18 (GPIO4/ADC1_CH4)
- net GPIO4: now also J3.11 (Pin_11)
- net GPIO5: now reaches U1.19 (GPIO5/ADC2_CH0)
- net GPIO5: now also J3.10 (Pin_10)
- net GPIO6: now reaches U1.20 (GPIO6)
- net GPIO6: now also J3.9 (Pin_9)
- net GPIO7: now reaches U1.21 (GPIO7)
- net GPIO7: now also J3.8 (Pin_8)
- net GPIO2: now reaches U1.5 (GPIO2/ADC1_CH2)
- net GPIO2: now also J2.4 (Pin_4)
- net GPIO3: now reaches U1.6 (GPIO3/ADC1_CH3)
- net GPIO3: now also J2.5 (Pin_5)
- net RXD renamed U0RXD
- net U0RXD: now also U2.21 (TXD), J3.3 (Pin_3); no longer U2.20 (RXD)
- net TXD renamed U0TXD
- net U0TXD: now also U2.20 (RXD), J3.2 (Pin_2); no longer U2.21 (TXD)
Other:
- note added: "CP2102"
- note added: "ESP32-C3-MINI-1"
- note added: "INPUTS AND OUTPUTS"
- moved on the sheet: C10, C11, C12, C13, C14, C15, C16, C2, C3, C4, C5, C6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
